File: ZodiarkSplit/ZodiarkSplit.sch (KiCad schematic (older format))
At the start: 130 parts, among them J2 MJ-4PP-9-Lily58-cache, P1 OLED, SW1 RST Button, SW2 Rotary_Encoder_Switch, U1 ProMicro, U10 HOLE-Lily58-cache, U2 HOLE-Lily58-cache, U3 HOLE-Lily58-cache, U4 HOLE-Lily58-cache, U5 HOLE-Lily58-cache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

Commit message: Final Proto
Parts:
- added LEFT5, LEFT6, LEFT7, LEFT8, RIGHT5, RIGHT6, RIGHT7, RIGHT8: JP1, Zodiark:Jumper, symbol Lily58-rescue:Jumper_NO_Small-Device
- added P2: OLED, Zodiark:OLED_4Pin, symbol Lily58-rescue:CONN_01X04-Lily58-cache
- added U11, U12, U13, U14: HOLE-Lily58-cache, Zodiark:HOLE_M2_TH, symbol Lily58-rescue:HOLE-Lily58-cache
- added U15, U16, U17, U18, U19, U20, U21: HOLE-Lily58-cache, Zodiark:HOLE_M2, symbol Lily58-rescue:HOLE-Lily58-cache
- LEFT1, LEFT2, LEFT3, LEFT4, RIGHT1, RIGHT2, RIGHT3, RIGHT4: footprint Jumper:SolderJumper-2_P1.3mm_Open_TrianglePad1.0x1.5mm -> Zodiark:Jumper
Connections:
- net GND: now also LEFT5.2, RIGHT8.2
- net SCL: now also LEFT7.2, RIGHT6.2
- net SDA: now also LEFT8.2, RIGHT5.2
- net VCC: now also LEFT6.2, RIGHT7.2
- new net: LEFT8.1, P2.1 (P1), RIGHT8.1
- new net: LEFT7.1, P2.2 (P2), RIGHT7.1
- new net: LEFT6.1, P2.3 (P3), RIGHT6.1
- new net: LEFT5.1, P2.4 (P4), RIGHT5.1
Other:
- moved on the sheet: U10
