File: ZodiarkSplit/Bottom Plate.kicad_pcb (KiCad board)
At the start: 2 copper layers, 159.7 x 129.2 mm, 13 parts

Commit message: Final Cleanup
Final Cleanup for public release.
Other:
- net class Default removed
- net class LED removed
- net class Power removed
