File: ZodiarkSplit/ZodiarkSplit.kicad_pcb (KiCad board)
At the start: 2 copper layers, 159.7 x 129.2 mm, 130 parts, among them J2 MJ-4PP-9-Lily58-cache, P1 OLED, SW1 RST Button, SW2 Rotary_Encoder_Switch, U1 ProMicro, U10 HOLE-Lily58-cache, U2 HOLE-Lily58-cache, U3 HOLE-Lily58-cache, U4 HOLE-Lily58-cache, U5 HOLE-Lily58-cache, U6 HOLE-Lily58-cache, U7 HOLE-Lily58-cache, U8 HOLE-Lily58-cache, U9 HOLE-Lily58-cache

Commit message: Final Proto
Parts:
- added LEFT5: JP1, Zodiark:Jumper, F.Cu at (177.4, 122.2)
- added LEFT6: JP1, Zodiark:Jumper, F.Cu at (174.8, 122.2)
- added LEFT7: JP1, Zodiark:Jumper, F.Cu at (172.2, 122.2)
- added LEFT8: JP1, Zodiark:Jumper, F.Cu at (169.7, 122.2)
- added P2: OLED, Zodiark:OLED_4Pin, F.Cu at (169.7, 124.6)
- added RIGHT5: JP1, Zodiark:Jumper, B.Cu at (177.4, 122.2)
- added RIGHT6: JP1, Zodiark:Jumper, B.Cu at (174.8, 122.2)
- added RIGHT7: JP1, Zodiark:Jumper, B.Cu at (172.2, 122.2)
- added RIGHT8: JP1, Zodiark:Jumper, B.Cu at (169.7, 122.2)
- added U11: HOLE-Lily58-cache, Zodiark:HOLE_M2_TH, F.Cu at (88.1, 139.1)
- added U12: HOLE-Lily58-cache, Zodiark:HOLE_M2_TH, F.Cu at (107.2, 140.2)
- added U13: HOLE-Lily58-cache, Zodiark:HOLE_M2_TH, F.Cu at (107.2, 101.8)
- added U14: HOLE-Lily58-cache, Zodiark:HOLE_M2_TH, F.Cu at (107.2, 64.0)
- added U15: HOLE-Lily58-cache, Zodiark:HOLE_M2, F.Cu at (145.4, 50.0)
- added U16: HOLE-Lily58-cache, Zodiark:HOLE_M2, F.Cu at (177.6, 83.6)
- added U17: HOLE-Lily58-cache, Zodiark:HOLE_M2, F.Cu at (169.6, 83.6)
- added U18: HOLE-Lily58-cache, Zodiark:HOLE_M2, F.Cu at (177.6, 127.5)
- added U19: HOLE-Lily58-cache, Zodiark:HOLE_M2, F.Cu at (173.8, 111.9)
- added U20: HOLE-Lily58-cache, Zodiark:HOLE_M2, F.Cu at (169.3, 127.5)
- added U21: HOLE-Lily58-cache, Zodiark:HOLE_M2, F.Cu at (173.8, 93.7)
- LEFT1, LEFT2, LEFT3, LEFT4, RIGHT1, RIGHT2, RIGHT3, RIGHT4: footprint Jumper:SolderJumper-2_P1.3mm_Open_TrianglePad1.0x1.5mm -> Zodiark:Jumper
- moved U5 125.4 mm to (50.0, 110.3)
- moved U2 75.0 mm to (175.7, 132.6)
- moved U3 45.1 mm to (126.2, 88.9)
- moved U9 42.3 mm to (88.1, 101.3)
- moved U8 22.6 mm to (88.3, 63.2)
- moved LEFT1 22.3 mm to (175.0, 61.9), turned to 180 degrees
- moved RIGHT1 22.3 mm to (175.0, 61.9), turned to 180 degrees
- moved LEFT2 19.3 mm to (175.0, 64.4), turned to 180 degrees
- moved RIGHT2 19.3 mm to (175.0, 64.4), turned to 180 degrees
- moved P1 17.3 mm to (177.3, 69.5), turned to 90 degrees
- moved LEFT3 16.7 mm to (175.0, 66.9), turned to 180 degrees
- moved RIGHT3 16.7 mm to (175.0, 66.9), turned to 180 degrees
- moved LEFT4 14.4 mm to (175.0, 69.5), turned to 180 degrees
- moved RIGHT4 14.4 mm to (175.0, 69.5), turned to 180 degrees
- moved SW1 7.99 mm to (177.3, 76.2)
Routing:
- net SCL: track 45.0 -> 96.5 mm, vias 5 -> 4
- net SDA: track 60.3 -> 103.8 mm, vias 6 -> 5
- net Net-(SW1-Pad1): track 37.9 -> 47.1 mm
- net VCC: track 1199.8 -> 1207.6 mm, vias 61 -> 63
- net ENC0: track 102.4 -> 107.4 mm
- net Net-(LEFT5-Pad1): track 0.00 -> 3.90 mm
- net Net-(LEFT6-Pad1): track 0.00 -> 3.89 mm
- net Net-(LEFT8-Pad1): track 0.00 -> 3.84 mm
- net Net-(LEFT7-Pad1): track 0.00 -> 3.74 mm
- net Net-(D62-Pad2): track 50.3 -> 47.7 mm
- net ROW3: track 253.3 -> 250.8 mm
- net GND: track 0.00 -> 2.05 mm
- net Net-(LEFT1-Pad1): track 5.10 -> 3.73 mm
- net Net-(LEFT2-Pad1): track 5.05 -> 3.72 mm
- net Net-(LEFT3-Pad1): track 5.00 -> 3.69 mm
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
Commit message: Final Cleanup
Final Cleanup for public release.
Parts:
- added G***: LOGO, Zodiark:Zodiark Logo, F.Cu at (156.2, 66.7)
- added G***: LOGO, Zodiark:Zodiark Logo, B.Cu at (155.7, 66.2)
- added REF**: MX_Kailh_Socket_Marks, Zodiark:MX_Kailh_Socket_Marks, F.Cu at (40.5, 69.8)
- added REF**: MX_Kailh_Socket_Marks, Zodiark:MX_Kailh_Socket_Marks, F.Cu at (97.6, 78.7)
- added REF**: MX_Kailh_Socket_Marks, Zodiark:MX_Kailh_Socket_Marks, F.Cu at (116.7, 81.8)
- added REF**: MX_Kailh_Socket_Marks, Zodiark:MX_Kailh_Socket_Marks, F.Cu at (135.7, 83.4)
- added REF**: MX_Kailh_Socket_Marks, Zodiark:MX_Kailh_Socket_Marks, F.Cu at (40.5, 108.0)
- added REF**: MX_Kailh_Socket_Marks, Zodiark:MX_Kailh_Socket_Marks, F.Cu at (59.5, 108.0)
- added REF**: MX_Kailh_Socket_Marks, Zodiark:MX_Kailh_Socket_Marks, F.Cu at (78.5, 100.2)
- added REF**: MX_Kailh_Socket_Marks, Zodiark:MX_Kailh_Socket_Marks, F.Cu at (97.7, 97.7)
- added REF**: MX_Kailh_Socket_Marks, Zodiark:MX_Kailh_Socket_Marks, F.Cu at (116.7, 100.8)
- added REF**: MX_Kailh_Socket_Marks, Zodiark:MX_Kailh_Socket_Marks, F.Cu at (135.7, 102.5)
- added REF**: MX_Kailh_Socket_Marks, Zodiark:MX_Kailh_Socket_Marks, F.Cu at (154.8, 92.9)
- added REF**: MX_Kailh_Socket_Marks, Zodiark:MX_Kailh_Socket_Marks, F.Cu at (59.6, 69.8)
- added REF**: MX_Kailh_Socket_Marks, Zodiark:MX_Kailh_Socket_Marks, F.Cu at (154.8, 112.0)
- added REF**: MX_Kailh_Socket_Marks, Zodiark:MX_Kailh_Socket_Marks, F.Cu at (135.7, 121.5)
- added REF**: MX_Kailh_Socket_Marks, Zodiark:MX_Kailh_Socket_Marks, F.Cu at (116.7, 119.8)
- added REF**: MX_Kailh_Socket_Marks, Zodiark:MX_Kailh_Socket_Marks, F.Cu at (97.7, 116.8)
- added REF**: MX_Kailh_Socket_Marks, Zodiark:MX_Kailh_Socket_Marks, F.Cu at (78.6, 119.2)
- added REF**: MX_Kailh_Socket_Marks, Zodiark:MX_Kailh_Socket_Marks, F.Cu at (59.5, 127.0)
- added REF**: MX_Kailh_Socket_Marks, Zodiark:MX_Kailh_Socket_Marks, F.Cu at (40.5, 127.1)
- added REF**: MX_Kailh_Socket_Marks, Zodiark:MX_Kailh_Socket_Marks, F.Cu at (40.5, 146.1)
- added REF**: MX_Kailh_Socket_Marks, Zodiark:MX_Kailh_Socket_Marks, F.Cu at (59.5, 146.1)
- added REF**: MX_Kailh_Socket_Marks, Zodiark:MX_Kailh_Socket_Marks, F.Cu at (78.5, 138.2)
- added REF**: MX_Kailh_Socket_Marks, Zodiark:MX_Kailh_Socket_Marks, F.Cu at (78.6, 62.0)
- added REF**: MX_Kailh_Socket_Marks, Zodiark:MX_Kailh_Socket_Marks, F.Cu at (97.6, 135.8)
- added REF**: MX_Kailh_Socket_Marks, Zodiark:MX_Kailh_Socket_Marks, F.Cu at (116.7, 138.9)
- added REF**: MX_Kailh_Socket_Marks, Zodiark:MX_Kailh_Socket_Marks, F.Cu at (143.7, 149.2)
- added REF**: MX_Kailh_Socket_Marks, Zodiark:MX_Kailh_Socket_Marks, F.Cu at (157.2, 134.9)
- added REF**: MX_Kailh_Socket_Marks, Zodiark:MX_Kailh_Socket_Marks, F.Cu at (164.3, 161.2)
- added REF**: MX_Kailh_Socket_Marks, Zodiark:MX_Kailh_Socket_Marks, F.Cu at (97.7, 59.6)
- added REF**: MX_Kailh_Socket_Marks, Zodiark:MX_Kailh_Socket_Marks, F.Cu at (116.7, 62.8)
- added REF**: MX_Kailh_Socket_Marks, Zodiark:MX_Kailh_Socket_Marks, F.Cu at (135.7, 64.3)
- added REF**: MX_Kailh_Socket_Marks, Zodiark:MX_Kailh_Socket_Marks, F.Cu at (40.5, 89.0)
- added REF**: MX_Kailh_Socket_Marks, Zodiark:MX_Kailh_Socket_Marks, F.Cu at (59.5, 89.0)
- added REF**: MX_Kailh_Socket_Marks, Zodiark:MX_Kailh_Socket_Marks, F.Cu at (78.6, 81.0)
Other:
- net class Default removed
- net class LED removed
- net class Power removed
- board text added: "By Split Logic Keyboards"
- board text added: "L00"
- board text added: "L01"
- board text added: "L02"
- board text added: "L03"
- board text added: "L04"
- board text added: "L05"
- board text added: "L06"
- board text added: "L10"
- board text added: "L11"
- board text added: "L12"
- board text added: "L13"
- board text added: "L14"
- board text added: "L15"
- board text added: "L16"
- board text added: "L20"
- board text added: "L21"
- board text added: "L22"
- board text added: "L23"
- board text added: "L24"
- board text added: "L25"
- board text added: "L26"
- board text added: "L30"
- board text added: "L31"
- board text added: "L32"
- board text added: "L33"
- board text added: "L34"
- board text added: "L35"
- board text added: "L36"
- board text added: "L40"
- board text added: "L41"
- board text added: "L42"
- board text added: "L43"
- board text added: "L44"
- board text added: "L45"
- board text added: "L46"
- board text added: "LED00"
- board text added: "LED01"
- board text added: "LED02"
- board text added: "LED03"
- board text added: "LED04"
- board text added: "LED05"
- board text added: "LED06"
- board text added: "LED07"
- board text added: "LED08"
- board text added: "LED09"
- board text added: "LED10"
- board text added: "LED11"
- board text added: "LED12"
- board text added: "LED13"
- board text added: "LED14"
- board text added: "LED15"
- board text added: "LED16"
- board text added: "LED17"
- board text added: "LED18"
- board text added: "LED19"
- board text added: "LED20"
- board text added: "LED21"
- board text added: "LED22"
- board text added: "LED23"
- board text added: "LED24"
- board text added: "LED25"
- board text added: "LED26"
- board text added: "LED27"
- board text added: "LED28"
- board text added: "LED29"
- board text added: "LED30"
- board text added: "LED31"
- board text added: "LED32"
- board text added: "LED33"
- board text added: "LED34"
- board text added: "LED35"
- board text added: "LED36"
- board text added: "LED37"
- board text added: "LED38"
- board text added: "LED39"
- board text added: "LED40"
- board text added: "LED41"
- board text added: "LED42"
- board text added: "LED43"
- board text added: "LED44"
- board text added: "LED45"
- board text added: "LED46"
- board text added: "LED47"
- board text added: "LED48"
- board text added: "LED49"
- board text added: "LED50"
- board text added: "LED51"
- board text added: "LED52"
- board text added: "LED53"
- board text added: "LED54"
- board text added: "LED55"
- board text added: "LED56"
- board text added: "LED57"
- board text added: "LED58"
- board text added: "LED59"
- board text added: "LED60"
- board text added: "LED61"
- board text added: "LED62"
- board text added: "LED63"
- board text added: "LED64"
- board text added: "LED65"
- board text added: "LED66"
- board text added: "LED67"
- board text added: "R00"
- board text added: "R01"
- board text added: "R02"
- board text added: "R03"
- board text added: "R04"
- board text added: "R05"
- board text added: "R06"
- board text added: "R10"
- board text added: "R11"
- board text added: "R12"
- board text added: "R13"
- board text added: "R14"
- board text added: "R15"
- board text added: "R16"
- board text added: "R20"
- board text added: "R21"
- board text added: "R22"
- board text added: "R23"
- board text added: "R24"
- board text added: "R25"
- board text added: "R26"
- board text added: "R30"
- board text added: "R31"
- board text added: "R32"
- board text added: "R33"
- board text added: "R34"
- board text added: "R35"
- board text added: "R36"
- board text added: "R40"
- board text added: "R41"
- board text added: "R42"
- board text added: "R43"
- board text added: "R44"
- board text added: "R45"
- board text added: "R46"
- board text added: "https://www.splitlogic.xyz/"
